File: Electrical/Power Distribution/Space Elevator Power Distributation Board/untitled.kicad_sch (KiCad schematic)
At the start: 11 parts, among them U3 MCP16361T-E_NMXVAO

Commit message: Changes to Power Distribution Schematic before PDR
Parts:
- added C10: 22u, symbol Device:C
- added C16, C17: 22uF, symbol Device:C
- added L2: L, symbol Device:L
- added U1: AP63203WU, Package_TO_SOT_SMD:TSOT-23-6, symbol Regulator_Switching:AP63203WU
- C9: value 22u -> 100nF
Connections:
- net +5V: now also C10.1, U1.2 (EN), U1.3 (IN)
- net +BATT: now also C6.1
- net GND: now also C5.2, C8.2, C10.2, C16.2, C17.2, U1.4 (GND); no longer C9.2
- net at C9.1: now also L2.1, U1.5 (SW); no longer C8.2
- new net: C9.2, U1.6 (BST)
- new net +3.3V: C16.1, C17.1, L2.2, U1.1 (FB)
Other:
- moved on the sheet: C5, C6, C7, C8, D3, L1, R14, R15, R16, U3
